File: hardware/SINSONTE_MODEL_B/SINSONTE_MODEL_B.kicad_pcb (KiCad board)
At the start: 2 copper layers, 90 x 70 mm, 43 parts, among them J1 BAT, J10 Conn_01x02_Male, J11 Conn_01x02_Male, J12 Conn_01x02_Male, J13 Conn_01x02_Male, J14 Conn_01x02_Male, J15 Conn_01x02_Male, J16 Conn_01x02_Male, J17 Conn_01x02_Male, J18 Conn_01x02_Male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

Commit message: shrinkikng in process
Parts:
- moved J13 36.0 mm to (117.0, 56.6), turned to 270 degrees
- moved R1 35.3 mm to (119.1, 77.0), turned to 0 degrees
- moved J12 33.7 mm to (117.0, 59.2), turned to 270 degrees
- moved J7 33.4 mm to (119.6, 56.6), turned to 0 degrees
- moved C1 33.0 mm to (123.5, 81.5)
- moved R2 32.8 mm to (119.5, 70.7)
- moved J11 31.7 mm to (117.0, 61.7), turned to 270 degrees
- moved J8 31.0 mm to (122.1, 56.6), turned to 0 degrees
- moved Q1 30.3 mm to (127.2, 74.0)
- moved J10 29.9 mm to (117.0, 64.3), turned to 270 degrees
- moved J18 28.9 mm to (124.7, 56.6), turned to 90 degrees
- moved J9 28.5 mm to (117.0, 66.8), turned to 270 degrees
- moved J17 26.0 mm to (124.7, 59.2), turned to 90 degrees
- moved J16 23.2 mm to (124.7, 61.7), turned to 90 degrees
- moved J15 20.8 mm to (124.7, 64.3), turned to 90 degrees
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Routing:
- net Net-(J8-Pad1): track 20.3 -> 0.00 mm
- net Net-(J7-Pad1): track 20.3 -> 0.00 mm
- net Net-(J6-Pad4): track 135.1 -> 128.8 mm
- net Net-(J9-Pad1): track 5.08 -> 0.00 mm
- net Net-(J13-Pad1): track 5.08 -> 0.00 mm
- net Net-(J12-Pad1): track 5.08 -> 0.00 mm
- net Net-(J11-Pad1): track 5.08 -> 0.00 mm
- net Net-(J10-Pad1): track 5.08 -> 0.00 mm
- net Net-(J18-Pad1): track 5.08 -> 0.00 mm
- net Net-(J17-Pad1): track 5.08 -> 0.00 mm
- net Net-(J16-Pad1): track 5.08 -> 0.00 mm
- net Net-(J15-Pad1): track 5.08 -> 0.00 mm
- net Net-(J14-Pad1): track 5.08 -> 0.00 mm
- net Net-(BT1-Pad1): track 125.3 -> 122.1 mm
- net Net-(J5-Pad19): track 37.4 -> 34.2 mm
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Other:
- outline, holes or cut-outs redrawn
- board text added: "+"
- board text added: "-"
- board text removed: "- +"

Commit message: shrinkikng finished
Parts:
- removed the G*** at (112.9, 79.5)
- removed the REF** at (108.1, 107.4)
- added REF**: OSHW-Symbol_6.7x6mm_SilkScreen, Symbol:OSHW-Symbol_6.7x6mm_SilkScreen, B.Cu at (132.2, 58.4)
- BT1: footprint Battery:BatteryHolder_Keystone_2462_2xAA -> Connector_PinHeader_2.54mm:PinHeader_1x02_P2.54mm_Vertical
- moved G*** 37.6 mm to (91.0, 86.3), turned to 0 degrees
- moved G*** 35.8 mm to (77.1, 72.3)
- moved REF** 29.0 mm to (136.0, 87.0)
- moved REF** 29.0 mm to (54.0, 87.0)
- moved J1 15.5 mm to (62.0, 86.8), turned to 0 degrees
- moved BT1 15.4 mm to (74.0, 86.4), turned to 90 degrees
- moved R3 5.88 mm to (127.9, 83.5)
- moved C1 5.38 mm to (118.4, 83.3)
Routing:
- net Net-(BT1-Pad2): track 312.6 -> 285.0 mm
- net Net-(BT1-Pad1): track 122.1 -> 114.2 mm
- net Net-(J2-Pad2): track 23.0 -> 26.7 mm
- net Net-(C1-Pad1): track 44.5 -> 47.3 mm
- net Net-(J5-Pad19): track 34.2 -> 31.5 mm
- net Net-(J6-Pad4): track 128.8 -> 126.8 mm
Other:
- board size 90 x 70 mm -> 90 x 41 mm
- board text added: "+ -"
- board text added: "MODEL B"
- board text removed: "MODEL A"
